File: eagle/TTS.sch (EAGLE design)
At the start: 14 parts, among them IC1 LM386N-1

Commit message: updates after build #1
Parts:
- C2, C3: device resistor:C-EU025-025X050 -> rcl:C-EU050-024X044
- R3: value 10k -> 10R
Connections:
- net N$2: now also R1.2, R2.1; no longer R1.1, R2.2
- net N$3: now also R2.2; no longer R1.2
- net N$7: now also R1.1; no longer R2.1
Other:
- moved on the sheet: R1, R2
Changed lines of the file:
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@@
 <setting verticaltext="up"/>
 </settings>
-<grid distance="0.1" unitdist="inch" unit="inch" style="lines" multiple="1" display="yes" altdistance="0.01" altunitdist="inch" altunit="inch"/>
+<grid distance="0.1" unitdist="inch" unit="inch" style="lines" multiple="1" display="no" altdistance="0.01" altunitdist="inch" altunit="inch"/>
 <layers>
 <layer number="1" name="Top" color="4" fill="1" visible="no" active="no"/>
@@
 <part name="IC1" library="linear" deviceset="LM386?-*" device="N" technology="1"/>
 <part name="C1" library="resistor" deviceset="C-EU" device="050-024X044" value="100n"/>
-<part name="C2" library="resistor" deviceset="C-EU" device="025-025X050" value="10n"/>
-<part name="C3" library="resistor" deviceset="C-EU" device="025-025X050" value="10n"/>
 <part name="C6" library="rcl" deviceset="CPOL-EU" device="E2.5-5" value="10u"/>
 <part name="C4" library="rcl" deviceset="CPOL-EU" device="E2.5-5" value="10u"/>
 <part name="C5" library="rcl" deviceset="CPOL-EU" device="E2.5-6" value="100u"/>
+<part name="R2" library="resistor" deviceset="R-EU_" device="0207/10" value="27k"/>
 <part name="R1" library="resistor" deviceset="R-EU_" device="0207/10" value="27k"/>
-<part name="R2" library="resistor" deviceset="R-EU_" device="0207/10" value="27k"/>
-<part name="R3" library="resistor" deviceset="R-EU_" device="0207/10" value="10k"/>
+<part name="R3" library="resistor" deviceset="R-EU_" device="0207/10" value="10R"/>
 <part name="JP1" library="pinhead" deviceset="PINHD-1X3" device="" value="In"/>
 <part name="JP2" library="pinhead" deviceset="PINHD-1X2" device="" value="Out"/>
@@
 <part name="R4" library="rcl" deviceset="POTENTIOMETER_" device="PT-10S" value="10k"/>
 <part name="C7" library="rcl" deviceset="CPOL-EU" device="E2.5-5" value="10u"/>
+<part name="C2" library="rcl" deviceset="C-EU" device="050-024X044" value="10n"/>
+<part name="C3" library="rcl" deviceset="C-EU" device="050-024X044" value="10n"/>
 </parts>
 <sheets>
@@
 <instance part="IC1" gate="G$1" x="43.18" y="68.58"/>
 <instance part="C1" gate="G$1" x="58.42" y="55.88"/>
-<instance part="C2" gate="G$1" x="-7.62" y="71.12"/>
-<instance part="C3" gate="G$1" x="7.62" y="71.12"/>
 <instance part="C6" gate="G$1" x="15.24" y="78.74" rot="R270"/>
 <instance part="C4" gate="G$1" x="45.72" y="58.42"/>
 <instance part="C5" gate="G$1" x="68.58" y="68.58" rot="R270"/>
-<instance part="R1" gate="G$1" x="0" y="78.74"/>
-<instance part="R2" gate="G$1" x="-15.24" y="78.74"/>
+<instance part="R2" gate="G$1" x="0" y="78.74"/>
+<instance part="R1" gate="G$1" x="-15.24" y="78.74"/>
 <instance part="R3" gate="G$1" x="58.42" y="63.5" rot="R90"/>
 <instance part="JP1" gate="A" x="-30.48" y="78.74" rot="R180"/>
@@
 <instance part="R4" gate="1" x="22.86" y="71.12" rot="R90"/>
 <instance part="C7" gate="G$1" x="48.26" y="78.74"/>
+<instance part="C2" gate="G$1" x="-7.62" y="71.12"/>
+<instance part="C3" gate="G$1" x="7.62" y="71.12"/>
 </instances>
 <busses>
@@
 </segment>
 </net>
-<net name="N$2" class="0">
+<net name="N$3" class="0">
 <segment>
 <pinref part="R2" gate="G$1" pin="2"/>
-<pinref part="R1" gate="G$1" pin="1"/>
-<wire x1="-10.16" y1="78.74" x2="-7.62" y2="78.74" width="0.1524" layer="91"/>
-<pinref part="C2" gate="G$1" pin="1"/>
-<wire x1="-7.62" y1="78.74" x2="-5.08" y2="78.74" width="0.1524" layer="91"/>
-<wire x1="-7.62" y1="73.66" x2="-7.62" y2="78.74" width="0.1524" layer="91"/>
-<junction x="-7.62" y="78.74"/>
-</segment>
-</net>
-<net name="N$3" class="0">
-<segment>
-<pinref part="R1" gate="G$1" pin="2"/>
 <pinref part="C6" gate="G$1" pin="-"/>
 <wire x1="5.08" y1="78.74" x2="7.62" y2="78.74" width="0.1524" layer="91"/>
-<pinref part="C3" gate="G$1" pin="1"/>
 <wire x1="7.62" y1="78.74" x2="10.16" y2="78.74" width="0.1524" layer="91"/>
 <wire x1="7.62" y1="73.66" x2="7.62" y2="78.74" width="0.1524" layer="91"/>
 <junction x="7.62" y="78.74"/>
+<pinref part="C3" gate="G$1" pin="1"/>
 </segment>
 </net>
@@
 <segment>
 <pinref part="JP1" gate="A" pin="2"/>
-<pinref part="R2" gate="G$1" pin="1"/>
+<pinref part="R1" gate="G$1" pin="1"/>
 <wire x1="-27.94" y1="78.74" x2="-20.32" y2="78.74" width="0.1524" layer="91"/>
 </segment>
@@
 <wire x1="58.42" y1="50.8" x2="76.2" y2="50.8" width="0.1524" layer="91"/>
 <wire x1="40.64" y1="60.96" x2="40.64" y2="50.8" width="0.1524" layer="91"/>
-<pinref part="C3" gate="G$1" pin="2"/>
 <wire x1="7.62" y1="66.04" x2="7.62" y2="50.8" width="0.1524" layer="91"/>
 <wire x1="7.62" y1="50.8" x2="22.86" y2="50.8" width="0.1524" layer="91"/>
-<pinref part="C2" gate="G$1" pin="2"/>
 <wire x1="22.86" y1="50.8" x2="35.56" y2="50.8" width="0.1524" layer="91"/>
 <wire x1="-7.62" y1="66.04" x2="-7.62" y2="50.8" width="0.1524" layer="91"/>
@@
 <pinref part="C1" gate="G$1" pin="2"/>
 <junction x="58.42" y="50.8"/>
+<pinref part="C2" gate="G$1" pin="2"/>
+<pinref part="C3" gate="G$1" pin="2"/>
 </segment>
 </net>
@@
 </segment>
 </net>
+<net name="N$2" class="0">
+<segment>
+<pinref part="R1" gate="G$1" pin="2"/>
+<pinref part="R2" gate="G$1" pin="1"/>
+<wire x1="-10.16" y1="78.74" x2="-7.62" y2="78.74" width="0.1524" layer="91"/>
+<pinref part="C2" gate="G$1" pin="1"/>
+<wire x1="-7.62" y1="78.74" x2="-5.08" y2="78.74" width="0.1524" layer="91"/>
+<wire x1="-7.62" y1="73.66" x2="-7.62" y2="78.74" width="0.1524" layer="91"/>
+<junction x="-7.62" y="78.74"/>
+</segment>
+</net>

Commit message: improve board labels
Parts:
- JP1: value In -> - In +
Changed lines of the file:
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@@
 <part name="R1" library="resistor" deviceset="R-EU_" device="0207/10" value="27k"/>
 <part name="R3" library="resistor" deviceset="R-EU_" device="0207/10" value="10R"/>
-<part name="JP1" library="pinhead" deviceset="PINHD-1X3" device="" value="In"/>
+<part name="JP1" library="pinhead" deviceset="PINHD-1X3" device="" value="- In +"/>
 <part name="JP2" library="pinhead" deviceset="PINHD-1X2" device="" value="Out"/>
 <part name="P+1" library="supply1" deviceset="VCC" device=""/>
